File: kicad_EPS_board/EPS/BMS.kicad_sch (KiCad schematic)
At the start: 13 parts, among them J2 UEXT, J3 USB_B_Micro, J4 Conn_01x04_Pin, J7 Conn_01x08_Pin

Commit message: kicad EPS board V2 revision and already generated html doc files
Connections:
- net +3V3 renamed +3.3V_BMS
Changed lines of the file:
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@@
 (kicad_sch
-	(version 20231120)
+	(version 20250114)
 	(generator "eeschema")
-	(generator_version "8.0")
+	(generator_version "9.0")
 	(paper "A4")
 	(junction
@@
 			)
 		)
-		(property "Value" "+3V3"
+		(property "Value" "+3.3V_BMS"
 			(at 220.091 47.6758 0)
 			(effects
@@
 		(at 161.29 49.53)
 		(size 35.56 55.88)
+		(exclude_from_sim no)
+		(in_bom yes)
+		(on_board yes)
+		(dnp no)
 		(fields_autoplaced yes)
 		(stroke
@@
 		(at 72.39 41.91)
 		(size 33.02 25.4)
+		(exclude_from_sim no)
+		(in_bom yes)
+		(on_board yes)
+		(dnp no)
 		(fields_autoplaced yes)
 		(stroke
@@
 		(at 166.37 125.73)
 		(size 22.86 15.24)
+		(exclude_from_sim no)
+		(in_bom yes)
+		(on_board yes)
+		(dnp no)
 		(fields_autoplaced yes)
 		(stroke
@@
 		(at 72.39 87.63)
 		(size 33.02 58.42)
+		(exclude_from_sim no)
+		(in_bom yes)
+		(on_board yes)
+		(dnp no)
 		(fields_autoplaced yes)
 		(stroke
