File: kicad_EPS_board/EPS/can.kicad_sch (KiCad schematic)
At the start: 10 parts, among them U6 TCAN334

Commit message: kicad EPS board V2 revision and already generated html doc files
Connections:
- net +3V3 renamed +3.3V_MPPT
