File: kicad_EPS_board/EPS/dcdc.kicad_sch (KiCad schematic)
At the start: 51 parts, among them Q1 IPA045N10N3G, Q2 IPA045N10N3G, Q3 IPA045N10N3G, U1 INA186, U2 LM5107

Commit message: kicad EPS board V2 revision and already generated html doc files
Parts:
- C47: renamed from C9; footprint LibreSolar:C_0805_2012 -> LibreSolar:C_0603_1608
- renumbered C1 to C39, C2 to C40, C3 to C41, C4 to C42, C5 to C43, C6 to C44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
Connections:
- net +3V3 renamed +3.3V_MPPT
