File: kicad_EPS_board/EPS/isl94202.kicad_sch (KiCad schematic)
At the start: 77 parts, among them Q10 BSS138, Q2 NDS0605, Q3 NDS0605, Q4 BSS138, Q5 BSS138, Q6 BSS138, Q7 BSS138, Q8 BSS138, Q9 NDS0605, U1 ISL94202

Commit message: kicad EPS board V2 revision and already generated html doc files
Connections:
- net +3V3 renamed +3.3V_BMS
Changed lines of the file:
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@@
 (kicad_sch
-	(version 20231120)
+	(version 20250114)
 	(generator "eeschema")
-	(generator_version "8.0")
+	(generator_version "9.0")
 	(paper "A4")
+	(text "Balancing (33R resistors)\nCurrent: 100-130 mA (3.3-4.2 V)\nHeat dissipation: 300-600 mW"
+		(exclude_from_sim no)
+		(at 119.38 190.5 0)
+		(effects
+			(font
+				(size 1.27 1.27)
+			)
+			(justify left bottom)
+		)
+	)
+	(text "On/off push button"
+		(exclude_from_sim no)
+		(at 220.98 20.32 0)
+		(effects
+			(font
+				(size 2.54 2.54)
+			)
+			(justify left bottom)
+		)
+	)
+	(text "ADDR pin low =\nI2C address 50H"
+		(exclude_from_sim no)
+		(at 156.21 130.81 0)
+		(effects
+			(font
+				(size 1.27 1.27)
+			)
+			(justify left bottom)
+		)
+	)
+	(text "Temperature sensors"
+		(exclude_from_sim no)
+		(at 205.74 119.38 0)
+		(effects
+			(font
+				(size 2.54 2.54)
+			)
+			(justify left bottom)
+		)
+	)
+	(text "Current sense filter"
+		(exclude_from_sim no)
+		(at 120.65 143.51 0)
+		(effects
+			(font
+				(size 2.54 2.54)
+			)
+			(justify left bottom)
+		)
+	)
 	(junction
 		(at 99.06 58.42)
@@
 		)
 	)
-	(text "Balancing (33R resistors)\nCurrent: 100-130 mA (3.3-4.2 V)\nHeat dissipation: 300-600 mW"
-		(exclude_from_sim no)
-		(at 119.38 190.5 0)
-		(effects
-			(font
-				(size 1.27 1.27)
-			)
-			(justify left bottom)
-		)
-	)
-	(text "On/off push button"
-		(exclude_from_sim no)
-		(at 220.98 20.32 0)
-		(effects
-			(font
-				(size 2.54 2.54)
-			)
-			(justify left bottom)
-		)
-	)
-	(text "ADDR pin low =\nI2C address 50H"
-		(exclude_from_sim no)
-		(at 156.21 130.81 0)
-		(effects
-			(font
-				(size 1.27 1.27)
-			)
-			(justify left bottom)
-		)
-	)
-	(text "Temperature sensors"
-		(exclude_from_sim no)
-		(at 205.74 119.38 0)
-		(effects
-			(font
-				(size 2.54 2.54)
-			)
-			(justify left bottom)
-		)
-	)
-	(text "Current sense filter"
-		(exclude_from_sim no)
-		(at 120.65 143.51 0)
-		(effects
-			(font
-				(size 2.54 2.54)
-			)
-			(justify left bottom)
-		)
-	)
 	(label "XT2"
 		(at 223.52 139.7 180)
@@
 			)
 		)
-		(property "Value" "+3V3"
+		(property "Value" "+3.3V_BMS"
 			(at 266.7 57.404 0)
 			(effects
