File: kicad_EPS_board/EPS/power_supply.kicad_sch (KiCad schematic)
At the start: 14 parts, among them U1 TPS560430X

Commit message: kicad EPS board V2 revision and already generated html doc files
Parts:
- renumbered C1 to C32, C2 to C33, C3 to C34, C4 to C35, C5 to C36, D1 to D11, D2 to D12, R1 to R72, R2 to R73, U1 to U5
Connections:
- net +3V3 renamed +3.3V_BMS
Changed lines of the file:
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@@
 (kicad_sch
-	(version 20231120)
+	(version 20250114)
 	(generator "eeschema")
-	(generator_version "8.0")
+	(generator_version "9.0")
 	(paper "A4")
+	(text "ToDo: Check Bourns inductor part number\n(L2) and possibly reduce footprint size"
+		(exclude_from_sim no)
+		(at 189.23 67.31 0)
+		(effects
+			(font
+				(size 1.27 1.27)
+			)
+			(justify left bottom)
+		)
+	)
+	(text "Battery to 3.3V (SMPS)"
+		(exclude_from_sim no)
+		(at 123.19 64.77 0)
+		(effects
+			(font
+				(size 2.54 2.54)
+			)
+			(justify left bottom)
+		)
+	)
+	(text "Vref = 1V"
+		(exclude_from_sim no)
+		(at 163.83 102.87 0)
+		(effects
+			(font
+				(size 1.27 1.27)
+			)
+			(justify left bottom)
+		)
+	)
 	(junction
 		(at 97.79 85.09)
@@
 			(width 0)
 			(type default)
-		)
-	)
-	(text "ToDo: Check Bourns inductor part number\n(L2) and possibly reduce footprint size"
-		(exclude_from_sim no)
-		(at 189.23 67.31 0)
-		(effects
-			(font
-				(size 1.27 1.27)
-			)
-			(justify left bottom)
-		)
-	)
-	(text "Battery to 3.3V (SMPS)"
-		(exclude_from_sim no)
-		(at 123.19 64.77 0)
-		(effects
-			(font
-				(size 2.54 2.54)
-			)
-			(justify left bottom)
-		)
-	)
-	(text "Vref = 1V"
-		(exclude_from_sim no)
-		(at 163.83 102.87 0)
-		(effects
-			(font
-				(size 1.27 1.27)
-			)
-			(justify left bottom)
 		)
 	)
@@
 		(on_board yes)
 		(dnp no)
-		(property "Reference" "#PWR04"
+		(property "Reference" "#PWR065"
 			(at 113.03 104.14 0)
 			(effects
@@
 		(on_board yes)
 		(dnp no)
-		(property "Reference" "C3"
+		(property "Reference" "C34"
 			(at 158.242 84.582 0)
 			(effects
@@
 		(on_board yes)
 		(dnp no)
-		(property "Reference" "#FLG01"
+		(property "Reference" "#FLG03"
 			(at 125.73 80.645 0)
 			(effects
@@
 		(on_board yes)
 		(dnp no)
-		(property "Reference" "C5"
+		(property "Reference" "C36"
 			(at 202.438 101.092 0)
 			(effects
@@
 		(on_board yes)
 		(dnp no)
-		(property "Reference" "#PWR09"
+		(property "Reference" "#PWR070"
 			(at 201.93 116.84 0)
 			(effects
@@
 		(on_board yes)
 		(dnp no)
-		(property "Reference" "C2"
+		(property "Reference" "C33"
 			(at 113.665 90.805 0)
 			(effects
@@
 		(on_board yes)
 		(dnp no)
-		(property "Reference" "R2"
+		(property "Reference" "R73"
 			(at 179.705 105.41 90)
 			(effects
@@
 		(on_board yes)
 		(dnp no)
-		(property "Reference" "U1"
+		(property "Reference" "U5"
 			(at 143.51 81.28 0)
 			(effects
@@
 		(on_board yes)
 		(dnp no)
-		(property "Reference" "#PWR01"
+		(property "Reference" "#PWR062"
 			(at 87.63 76.2 0)
 			(effects
@@
 		(on_board yes)
 		(dnp no)
-		(property "Reference" "#FLG02"
+		(property "Reference" "#FLG04"
 			(at 186.69 85.725 0)
 			(effects
@@
 		(on_board yes)
 		(dnp no)
-		(property "Reference" "C1"
+		(property "Reference" "C32"
 			(at 98.425 90.805 0)
 			(effects
@@
 		(on_board yes)
 		(dnp no)
-		(property "Reference" "#PWR05"
+		(property "Reference" "#PWR066"
 			(at 130.81 104.14 0)
 			(effects
@@
 		(on_board yes)
 		(dnp no)
-		(property "Reference" "#PWR06"
+		(property "Reference" "#PWR067"
 			(at 181.61 116.84 0)
 			(effects
@@
 		(on_board yes)
 		(dnp no)
-		(property "Reference" "#PWR07"
+		(property "Reference" "#PWR068"
 			(at 191.77 116.84 0)
 			(effects
@@
 		(on_board yes)
 		(dnp no)
-		(property "Reference" "#PWR03"
+		(property "Reference" "#PWR064"
 			(at 97.79 104.14 0)
 			(effects
@@
 		(on_board yes)
 		(dnp no)
-		(property "Reference" "C4"
+		(property "Reference" "C35"
 			(at 192.278 101.092 0)
 			(effects
@@
 		(on_board yes)
 		(dnp no)
-		(property "Reference" "D2"
+		(property "Reference" "D12"
 			(at 77.47 115.1636 0)
 			(effects
@@
 		(on_board yes)
 		(dnp no)
-		(property "Reference" "D1"
+		(property "Reference" "D11"
 			(at 77.47 69.4436 0)
 			(effects
@@
 		(on_board yes)
 		(dnp no)
-		(property "Reference" "R1"
+		(property "Reference" "R72"
 			(at 179.705 95.25 90)
 			(effects
@@
 		(on_board yes)
 		(dnp no)
-		(property "Reference" "#PWR08"
+		(property "Reference" "#PWR069"
 			(at 201.93 91.44 0)
 			(effects
@@
 			)
 		)
-		(property "Value" "+3V3"
+		(property "Value" "+3.3V_BMS"
 			(at 201.93 84.074 0)
 			(effects
@@
 		(on_board yes)
 		(dnp no)
-		(property "Reference" "#PWR02"
+		(property "Reference" "#PWR063"
 			(at 87.63 121.92 0)
 			(effects
